Commit message: fix problems

File: baxter_vision_example/urdf/baxter.urdf (robot description, URDF)
Before this commit: robot baxter, 54 links, 53 joints
Links:
- removed link xtion_depth_frame
- removed link xtion_depth_optical_frame
- removed link xtion_link
- removed link xtion_rgb_frame
- removed link xtion_rgb_optical_frame
Joints:
- removed joint xtion_depth_joint
- removed joint xtion_depth_optical_joint
- removed joint xtion_joint
- removed joint xtion_rgb_joint
- removed joint xtion_rgb_optical_joint

File: baxter_vision_example/urdf/baxter.xacro (robot description, xacro)
@@ -9,4 +9,74 @@
   <xacro:property name="right_wrist_offset_x" value="-0.01" />
   <xacro:property name="left_wrist_offset_x" value="-0.01" />
+  <!-- kinect-->
+  <joint name="xtion_joint" type="fixed">
+    <origin rpy="0 0 0" xyz="-0.069 0.0 0.263"/>
+    <parent link="head"/>
+    <child link="xtion_link"/>
+  </joint>
+  <link name="xtion_link">
+    <inertial>
+      <mass value="0.200"/>
+      <origin rpy="0 0 0" xyz="0 0 0"/>
+      <inertia ixx="5.8083e-4" ixy="0" ixz="0" iyy="3.0833e-5" iyz="0" izz="5.9083e-4"/>
+    </inertial>
+  </link>
+  <joint name="xtion_depth_joint" type="fixed">
+    <origin rpy="0 0 0" xyz="0.0 0.049 0.0"/>
+    <parent link="xtion_link"/>
+    <child link="xtion_depth_frame"/>
+  </joint>
+  <link name="xtion_depth_frame"/>
+  <joint name="xtion_depth_optical_joint" type="fixed">
+    <origin rpy="-1.57079632679 0.0 -1.57079632679" xyz="0 0 0"/>
+    <parent link="xtion_depth_frame"/>
+    <child link="xtion_depth_optical_frame"/>
+  </joint>
+  <link name="xtion_depth_optical_frame"/>
+  <joint name="xtion_rgb_joint" type="fixed">
+    <origin rpy="0 0 0" xyz="0.0 0.022 0.0"/>
+    <parent link="xtion_link"/>
+    <child link="xtion_rgb_frame"/>
+  </joint>
+  <link name="xtion_rgb_frame"/>
+  <joint name="xtion_rgb_optical_joint" type="fixed">
+    <origin rpy="-1.57079632679 0.0 -1.57079632679" xyz="0 0 0"/>
+    <parent link="xtion_rgb_frame"/>
+    <child link="xtion_rgb_optical_frame"/>
+  </joint>
+  <link name="xtion_rgb_optical_frame"/>
+  <gazebo reference="xtion_depth_frame">
+    <sensor name="xtion" type="depth">
+      <update_rate>20</update_rate>
+      <camera>
+        <horizontal_fov>1.09606677025</horizontal_fov>
+        <image>
+          <format>R8G8B8</format>
+          <width>640</width>
+          <height>480</height>
+        </image>
+        <clip>
+          <near>0.5</near>
+          <far>9</far>
+        </clip>
+      </camera>
+      <plugin filename="libgazebo_ros_openni_kinect.so" name="xtion_camera_controller">
+        <alwaysOn>true</alwaysOn>
+        <updateRate>20</updateRate>
+        <imageTopicName>xtion/rgb/image_raw</imageTopicName>
+        <cameraInfoTopicName>xtion/rgb/camera_info</cameraInfoTopicName>
+        <depthImageTopicName>xtion/depth/image_raw</depthImageTopicName>
+        <depthImageCameraInfoTopicName>xtion/depth/camera_info</depthImageCameraInfoTopicName>
+        <pointCloudTopicName>xtion/depth/points</pointCloudTopicName>
+        <frameName>xtion_depth_optical_frame</frameName>
+        <distortion_k1>0.0</distortion_k1>
+        <distortion_k2>0.0</distortion_k2>
+        <distortion_k3>0.0</distortion_k3>
+        <distortion_t1>0.0</distortion_t1>
+        <distortion_t2>0.0</distortion_t2>
+      </plugin>
+    </sensor>
+  </gazebo>
+  <!-- kinect-->
   <!-- custom vacuum gripper >>>>>>>>>>>>>>>>>>>>>>>>>>>>>>>>>>>>>>>>>>>>>>>>>> -->
   <link name="right_custom_vacuum_link">
